File: hat-fuji-41d/hat-fuji-41d.kicad_pcb (KiCad board)
At the start: 2 copper layers, 87.4 x 55.4 mm, 28 parts, among them J1 Conn_02x10_Odd_Even, J2 Conn_01x20_Pin, J3 Conn_01x20_Pin, J4 Conn_02x04_Odd_Even, P2 ST-TF-003A, SW2 K2-1808SN-A4SW-01, SW3 K2-1808SN-A4SW-01, U2 ESP32-DevKitC-VE

Commit message: add hat-fuji-41d kicad & gerbers.
Routing:
- net +3.3V: track 228.1 -> 254.7 mm
- net Net-(J3-Pin_18): track 28.4 -> 20.5 mm
- net /H12: track 128.3 -> 125.6 mm
Other:
- board text added: "41d"
- board text added: "Special Thanks to * Bill Athing * Andy Diller"
- board text added: "[ n*n + n + 41 for n in range(40) ]"
- board text added: "lambda n: n > and all(n % d for d in range(2, n))"
- board text removed: "Special Thanks to * Bill Athing * MassiveRobot"
- board text removed: "ยอ ยักษ์"
