File: hat-fuji-41d/hat-fuji-41d.kicad_sch (KiCad schematic)
At the start: 28 parts, among them J1 Conn_02x10_Odd_Even, J2 Conn_01x20_Pin, J3 Conn_01x20_Pin, J4 Conn_02x04_Odd_Even, P2 ST-TF-003A, SW2 K2-1808SN-A4SW-01, SW3 K2-1808SN-A4SW-01, U2 ESP32-DevKitC-VE

Commit message: add hat-fuji-41d kicad & gerbers.
Other:
- company: (none) -> Copico Labs
- title: CoCo FujiNet -> FujiNet Hat rev 41d for centipede 32z and TFR/911h
Changed lines of the file:
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@@
 	(paper "A4")
 	(title_block
-		(title "CoCo FujiNet")
-		(date "2024-08-25")
-		(rev "Rev 0000")
+		(title "FujiNet Hat rev 41d for centipede 32z and TFR/911h")
+		(date "2026-10-19")
+		(rev "41d")
+		(company "Copico Labs")
 	)
 	(text "50A PowerDI-123\nSchottky Diode"
